File: satellite_watch/mb.kicad_sch (KiCad schematic)
At the start: 49 parts, among them J1 PogoPins_02x17_Data, J2 UJ20-C-H-G-MSMT-2B-P16-TR, J5 Pogo_02x03_Power, Q2 Q_NMOS_Depletion_DGS, Q3 DMP1045U, Q4 Q_NMOS_Depletion_DGS, SW1 B3U-1000P, SW2 B3U-1000P, SW3 B3U-1000P, SW4 B3U-1000P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

Commit message: v0.15
wip of large-size PCB
Parts:
- removed BT1: CR1220, symbol Device:Battery_Cell
- added BT3: 2895 (CR1220 Holder), footprint:BAT_2895, symbol import_symbol:2895
- added C16: 10uF, Capacitor_SMD:C_0603_1608Metric_Pad1.08x0.95mm_HandSolder, symbol Device:C_Small
- added C17: 22uF, Capacitor_SMD:C_0603_1608Metric_Pad1.08x0.95mm_HandSolder, symbol Device:C_Small
- added L1: 2.2Uh, Inductor_SMD:L_0603_1608Metric_Pad1.05x0.95mm_HandSolder, symbol Device:L_Small
- added R19, R20: 2.2K, Resistor_SMD:R_0603_1608Metric_Pad0.98x0.95mm_HandSolder, symbol Device:R_Small_US
- added R21: 100K, Resistor_SMD:R_0603_1608Metric_Pad0.98x0.95mm_HandSolder, symbol Device:R_Small_US
- added R3: 750K, Resistor_SMD:R_0603_1608Metric_Pad0.98x0.95mm_HandSolder, symbol Device:R_Small_US
- added TP3: BAT+, TestPoint:TestPoint_Pad_D2.5mm, symbol Connector:TestPoint
- added TP4: BAT-, TestPoint:TestPoint_Pad_D2.5mm, symbol Connector:TestPoint
- added U7: PAM2401SCADJ, footprint:MSOP8_DIO, symbol import_symbol:PAM2401SCADJ
- C1, C10, C11, C12, C13, C14, C15, C2, C3, C4, C6, C7, C8, C9: footprint (none) -> Capacitor_SMD:C_0603_1608Metric_Pad1.08x0.95mm_HandSolder
- D1: footprint Diode_SMD:D_SMA -> Diode_SMD:D_0603_1608Metric_Pad1.05x0.95mm_HandSolder
- D2, D3: footprint (none) -> LED_SMD:LED_0603_1608Metric_Pad1.05x0.95mm_HandSolder
- J1: footprint (none) -> Connector_PinHeader_2.54mm:PinHeader_2x17_P2.54mm_Vertical
- J2: footprint UJ20-C-H-G-MSMT-2B-P16-TR:SAMESKY_UJ20-C-H-G-MSMT-2B-P16-TR -> footprint:SAMESKY_UJ20-C-H-G-MSMT-2B-P16-TR
- J5: footprint (none) -> Connector_PinHeader_2.54mm:PinHeader_2x03_P2.54mm_Vertical
- Q2, Q4: value Q_NMOS_Depletion_DGS -> BSS138; footprint (none) -> Package_TO_SOT_SMD:SOT-23-3
- Q3: footprint DMP1045U:SOT91P240X110-3N -> Package_TO_SOT_SMD:SOT-23-3
- R1, R10, R11, R12, R13, R14, R15, R16, R17, R18, R2, R4, R5, R8, R9: footprint (none) -> Resistor_SMD:R_0603_1608Metric_Pad0.98x0.95mm_HandSolder
- SW1, SW2, SW3, SW4, SW5: footprint (none) -> Button_Switch_SMD:SW_SPST_B3U-1000P
- U2: footprint MAX30101EFD_T:PSON80P560X330X165-14N -> footprint:PSON80P560X330X165-14N
- U4: footprint NCP186AMX330TAG:PSON40P160X120X45-9N -> footprint:PSON40P160X120X45-9N
Connections:
- net BAT+: now also TP3.1
- net BAT-: now also TP4.1
- net GND: now also BT3.N, C16.2, C17.2, R21.2, U7.4 (AGND), U7.8 (PGND)
- net GPIO5/SDA: now also R20.2
- net GPIO6/SCL: now also R19.2
- net VCC_3V3: now also C16.1, L1.1, R19.1, R20.1, U7.2 (EN), U7.3 (VIN); no longer C7.1, R10.1, U4.1 (OUT), U4.2 (OUT__1), U4.4 (FB/ADJ)
- net at U5.6 (VBAT): now also BT3.P1, BT3.P2
- net VCC_5V renamed VUSB_5V
- net VUSB_5V: no longer C9.1, D1.2 (A), Q3.1, R9.1, U2.10 (VLED+__1), U2.9 (VLED+)
- new net: R21.1, R3.1, U7.5 (FB)
- new net: L1.2, U7.1 (LX)
- new net IC_5V: C17.1, C9.1, R3.2, U2.10 (VLED+__1), U2.9 (VLED+), U7.7 (OUT)
- new net VIN_3V3: C7.1, D1.2 (A), Q3.1, R10.1, R9.1, U4.1 (OUT), U4.2 (OUT__1), U4.4 (FB/ADJ)
- no-connect marks 3 -> 4
Other:
- note added: "DC-DC CONVERTER TO 5V FOR MAX30101 INPUT: 2.4-4.75V"
- moved on the sheet: D1, J1, J5, Q3, R8, R9
