File: schematics/satWatch_main_LargePrototype/satWatch_main_LargePrototype.kicad_sch (KiCad schematic)
At the start: 102 parts, among them J1 PogoPins_02x17_Data, J2 UJ20-C-H-G-MSMT-2B-P16-TR, J5 Pogo_02x03_Power, Q1 FS8205, Q2 BSS138, Q3 DMP1045U, Q4 BSS138, SW1 B3U-1000P, SW2 B3U-1000P, SW3 B3U-1000P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

Commit message: v0.3
Finalized initial draft of large mainboard PCB, ready for first production and testing
Parts:
- added C24, C25: 22pF, Capacitor_SMD:C_0603_1608Metric_Pad1.08x0.95mm_HandSolder, symbol Device:C_Small
- added C26, C27: 0.1uF, Capacitor_SMD:C_0603_1608Metric_Pad1.08x0.95mm_HandSolder, symbol Device:C_Small
- added R26, R6: 10K, Resistor_SMD:R_0603_1608Metric_Pad0.98x0.95mm_HandSolder, symbol Device:R_Small_US
- added R32, R33: 0, Resistor_SMD:R_0603_1608Metric_Pad0.98x0.95mm_HandSolder, symbol Device:R_Small_US
- added TP23: PPG_MISO, TestPoint:TestPoint_Pad_D2.5mm, symbol Connector:TestPoint
- added TP24: PPG_MOSI, TestPoint:TestPoint_Pad_D2.5mm, symbol Connector:TestPoint
- added TP25: PPG_SCK, TestPoint:TestPoint_Pad_D2.5mm, symbol Connector:TestPoint
- added TP26: PPG_CSB, TestPoint:TestPoint_Pad_D2.5mm, symbol Connector:TestPoint
- added TP27: PPG_INT, TestPoint:TestPoint_Pad_D2.5mm, symbol Connector:TestPoint
- added U12: BNO085, footprint:IC_BNO085, symbol symbols:BNO085
- added Y2: 32.768Hz, footprint:ABS07-32.768KHZ-T, symbol Device:Crystal
- C10, C21, C22, C23, C5, C9: footprint (none) -> Capacitor_SMD:C_0603_1608Metric_Pad1.08x0.95mm_HandSolder
- LED1: footprint SFH 7013_OSR -> footprint:SFH7016
- R27, R28, R29, R30, R31: footprint (none) -> Resistor_SMD:R_0603_1608Metric_Pad0.98x0.95mm_HandSolder
- U10, U11: footprint 6p550-5354p01-4_VIS -> footprint:VEMD8080
- U2: footprint 21-100134A_20_MXM -> footprint:MAX86141ENP
- U3: footprint 21-100264_T2433+2C_MXM -> footprint:MAX32664GTGB+T
- Y1: value 32.768kHz, 6pF (CM1610H32768DZB) -> 32.768kHz; footprint (none) -> footprint:ABS07-32.768KHZ-T
Connections:
- net MCU_MFIO is gone; now on net GPIO11: U3.1 (MFIO)
- net MCU_RSTN is gone; now on net GPIO10: C23.1, U3.6 (RSTN)
- net GND: now also C24.2, C25.2, C26.2, C27.2, R26.1, R6.1, U12.10 (CLKSEL0), U12.2 (GND), U12.25 (GNDIO)
- net GPIO33: now also J1.18 (Pin_18); no longer J1.17 (Pin_17)
- net GPIO34: now also J1.19 (Pin_19); no longer J1.34 (Pin_34)
- net GPIO35: now also J1.21 (Pin_21); no longer J1.33 (Pin_33)
- net GPIO36: now also J1.22 (Pin_22); no longer J1.32 (Pin_32)
- net GPIO37: now also J1.23 (Pin_23); no longer J1.31 (Pin_31)
- net GPIO38: now also J1.24 (Pin_24); no longer J1.30 (Pin_30)
- net GPIO39: now also J1.25 (Pin_25); no longer J1.29 (Pin_29)
- net GPIO40: now also J1.26 (Pin_26); no longer J1.28 (Pin_28)
- net GPIO42: now also J1.28 (Pin_28); no longer J1.26 (Pin_26)
- net GPIO45: now also J1.31 (Pin_31); no longer J1.25 (Pin_25)
- net GPIO46: now also J1.32 (Pin_32); no longer J1.24 (Pin_24)
- net GPIO47: now also J1.17 (Pin_17); no longer J1.23 (Pin_23)
- net GPIO48: now also J1.20 (Pin_20); no longer J1.22 (Pin_22)
- net GPIO5/SDA: now also U12.20 (H_SDA/H_MISO/TX)
- net GPIO6/SCL: now also U12.19 (H_SCL/SCK/RX)
- net LV_SCL: now also J1.34 (Pin_34); no longer J1.19 (Pin_19)
- net LV_SDA: now also J1.33 (Pin_33); no longer J1.18 (Pin_18)
- net PPG_CSB: now also TP26.1
- net PPG_INT: now also TP27.1
- net PPG_MISO: now also TP23.1
- net PPG_MOSI: now also TP24.1
- net PPG_SCK: now also TP25.1
- net U0RXD: now also J1.30 (Pin_30); no longer J1.20 (Pin_20)
- net U0TXD: now also J1.29 (Pin_29); no longer J1.21 (Pin_21)
- net VCC_3V3: now also C27.1, R32.2, R33.1, U12.28 (VDDIO), U12.3 (VDD)
- new net: U12.1 (RESV_NC), U12.12 (RESV_NC), U12.13 (RESV_NC), U12.21 (RESV_NC), U12.22 (RESV_NC), U12.23 (RESV_NC), U12.24 (RESV_NC), U12.7 (RESV_NC), U12.8 (RESV_NC)
- new net: C24.1, U12.26 (XOUT32/CLKSEL1), Y2.2
- new net: C25.1, U12.27 (XIN32), Y2.1
- new net: C26.1, U12.9 (CAP)
- new net ACCEL_BOOT: U12.4 (~{BOOT})
- new net ACCEL_CS: U12.18 (~{H_CS})
- new net ACCEL_INT: U12.14 (~{H_INT})
- new net ACCEL_MOSI: U12.17 (SA0/H_MOSI)
- new net ACCEL_PS0: R26.2, R33.2, U12.6 (PS0/WAKE)
- new net ACCEL_PS1: R32.1, R6.2, U12.5 (PS1)
- new net ACCEL_RST: U12.11 (~{RST})
- no-connect marks 9 -> 11
Other:
- note removed: "9 AXIS IMU BMO085"
