File: schematics/satWatch_main_LargePrototype/satWatch_main_LargePrototype.kicad_sch (KiCad schematic)
At the start: 120 parts, among them J1 PogoPins_02x17_Data, J2 UJ20-C-H-G-MSMT-2B-P16-TR, J5 Pogo_02x03_Power, Q1 FS8205, Q2 BSS138, Q3 DMP1045U, Q4 BSS138, SW1 B3U-1000P, SW2 B3U-1000P, SW3 B3U-1000P, SW4 B3U-1000P, SW5 B3U-1000P, U1 ESP32-S3-MINI-1, U10 VEMD8080, U11 VEMD8080, U12 BNO085, U2 MAX86141, U3 MAX32664GTGC, U4 NCP186AMX330TAG, U5 DS3231MZ, U6 MIC5365-1.8YC5, U7 PAM2401SCADJ, U8 TP4056-42-ESOP8, U9 DW01A, Y1 32.768kHz, Y2 32.768Hz

Commit message: v0.5
removed MAX3264/MAX86141 for MAX30101 for reduced scope. editted PCB and via sizes based on manufacturer response.
Parts:
- removed C10, C29: 0.1uF, Capacitor_SMD:C_0603_1608Metric_Pad1.08x0.95mm_HandSolder, symbol Device:C_Small
- removed C23: 1uF, Capacitor_SMD:C_0603_1608Metric_Pad1.08x0.95mm_HandSolder, symbol Device:C_Small
- removed C28: 22uF, Capacitor_SMD:C_0603_1608Metric_Pad1.08x0.95mm_HandSolder, symbol Device:C_Small
- removed C5, C9: 10uF, Capacitor_SMD:C_0603_1608Metric_Pad1.08x0.95mm_HandSolder, symbol Device:C_Small
- removed LED1: SFH 7016, footprint:SFH7016, symbol symbols:SFH_7013
- removed NT1: NetTie_2, NetTie:NetTie-2_SMD_Pad0.5mm, symbol Device:NetTie_2
- removed R28: 100K, Resistor_SMD:R_0603_1608Metric_Pad0.98x0.95mm_HandSolder, symbol Device:R_Small_US
- removed R29, R30, R31: 0, Resistor_SMD:R_0603_1608Metric_Pad0.98x0.95mm_HandSolder, symbol Device:R_Small_US
- removed TP23: PPG_MISO, TestPoint:TestPoint_Pad_D2.5mm, symbol Connector:TestPoint
- removed TP24: PPG_MOSI, TestPoint:TestPoint_Pad_D2.5mm, symbol Connector:TestPoint
- removed TP25: PPG_SCK, TestPoint:TestPoint_Pad_D2.5mm, symbol Connector:TestPoint
- removed TP26: PPG_CSB, TestPoint:TestPoint_Pad_D2.5mm, symbol Connector:TestPoint
- removed TP27: PPG_INT, TestPoint:TestPoint_Pad_D2.5mm, symbol Connector:TestPoint
- removed U10, U11: VEMD8080, footprint:VEMD8080, symbol symbols:VEMD8080
- removed U2: MAX86141, footprint:MAX86141ENP, symbol symbols:MAX86141ENP+
- removed U3: MAX32664GTGC, footprint:MAX32664GTGB+T, symbol symbols:MAX32664GTGB+T
- removed Y1: 32.768kHz, footprint:ABS07-32.768KHZ-T, symbol Device:Crystal
- added U2: MAX30101EFD_T, footprint:MAX30101EFD+T, symbol symbols:MAX30101EFD_T
- C21: value 1uF -> 10uF
- C22: value 1uF -> 0.1uF
- R27: value 10 -> 4.7K
Connections:
- net VCC_1V8 is gone; now on net 1V8: J5.4 (Pin_4), Q2.2 (G), Q4.2 (G), R12.1, R13.1
- net VUSB_5V is gone; now on net USB_5V: C18.1, D6.2 (A), D7.2 (A), U8.4 (V_{CC}), U8.8 (CE)
- net 1V8: now also C22.1, U2.11 (VDD); no longer C21.1
- net 5V: now also C21.1, U2.10 (VLED+__1), U2.9 (VLED+)
- net GND: now also U2.12 (GND), U2.4 (PGND); no longer R27.2
- net LV_SCL: now also U2.2 (SCL)
- net LV_SDA: now also U2.3 (SDA)
- net VCC_3V3: now also R27.2
- net at R27.1: now also U2.13 (~{INT})
- no-connect marks 11 -> 7
Other:
- note added: "REFERENCE DESIGN FROM SPARKFUN MAX30101 QWIC TYPICAL CURRENT CONSUMPTION 600-1000uA VCC RANGE: 1.7 - 2.0V VCC RED/IR LED: 3.1-5.0V VCC GREN LED: 4.5-5.5V I2C ADD: 0X57"
- note removed: "GROUND LINE ROUTES SEPERATELY FROM PHOTODIODE PAD & MAIN GROUND"
- note removed: "LED1 = GREEN 530nm LED2 = IR 90nm LED3 = RED 655nm"
- note removed: "REFERENCE DESIGN FROM ANALOGDEVICES - MAXREFDES103 - SENSOR HUB REQUIRES ACCELEROMETER DATA: WILL BE FED FROM HOST-SIDE"
- moved on the sheet: BT3, C1, C11, C12, C13, C14, C15, C16, C17, C18, C19, C2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
