File: schematics/satWatch_main/satWatch_face1.kicad_sch (KiCad schematic)
At the start: 0 parts

Commit message: v1.1
Completed board layout for charging dock configuration and a default watchface config
Parts:
- added C33: 1uF, Capacitor_SMD:C_0402_1005Metric_Pad0.74x0.62mm_HandSolder, symbol Device:C_Small
- added C34: 0.1uF, Capacitor_SMD:C_0402_1005Metric_Pad0.74x0.62mm_HandSolder, symbol Device:C_Small
- added D11, D12, D13, D14, D15, D16, D17, D18: LED, LED_SMD:LED_1206_3216Metric_Pad1.42x1.75mm_HandSolder, symbol Device:LED
- added J10: BAT+, Connector_Wire:SolderWirePad_1x01_SMD_3x6mm, symbol Connector:Conn_01x01_Pin
- added J11: BAT-, Connector_Wire:SolderWirePad_1x01_SMD_3x6mm, symbol Connector:Conn_01x01_Pin
- added J7: 2167010509_MOLEX, footprint:CON_2167010509_MOL, symbol Connector_Generic:Conn_02x25_Top_Bottom
- added J8: MOTOR+, Connector_Wire:SolderWirePad_1x01_SMD_3x6mm, symbol Connector:Conn_01x01_Pin
- added J9: MOTOR-, Connector_Wire:SolderWirePad_1x01_SMD_3x6mm, symbol Connector:Conn_01x01_Pin
- added Q6: MMBT2222A, Package_TO_SOT_SMD:SOT-23, symbol Transistor_BJT:MMBT2222A
- added Q7: FS8205, footprint:SOT95P280X145-6N, symbol symbols:FS8205
- added R33: 1K, Resistor_SMD:R_0402_1005Metric_Pad0.72x0.64mm_HandSolder, symbol Device:R_Small_US
- added R34: 22, Resistor_SMD:R_0402_1005Metric_Pad0.72x0.64mm_HandSolder, symbol Device:R_Small_US
- added R35, R36, R47, R48, R49, R50: 10K, Resistor_SMD:R_0402_1005Metric_Pad0.72x0.64mm_HandSolder, symbol Device:R_Small_US
- added R37, R38, R39, R40, R41, R42, R43, R44: 180, Resistor_SMD:R_0402_1005Metric_Pad0.72x0.64mm_HandSolder, symbol Device:R_Small_US
- added R45: 100, Resistor_SMD:R_0402_1005Metric_Pad0.72x0.64mm_HandSolder, symbol Device:R_US
- added R46: 1K, Resistor_SMD:R_0402_1005Metric_Pad0.72x0.64mm_HandSolder, symbol Device:R_US
- added U11: (no value), footprint:Wisevision N096-1608TBBIG11-H13, symbol symbols:N096-1608TBBIG11-H13
- added U12: (no value), Package_TO_SOT_SMD:SOT-23, symbol symbols:APX803
- added U13: DRV2605LDGS, Package_SO:TSSOP-10_3x3mm_P0.5mm, symbol Driver:DRV2605LDGS
- added U14: DW01A, Package_TO_SOT_SMD:SOT-23-6, symbol Battery_Management:DW01A
Connections:
- new net: D18.2 (A), R44.1
- new net: D16.2 (A), R42.1
- new net: D14.2 (A), R40.1
- new net: J9.1 (Pin_1), U13.9 (OUT-)
- new net: Q6.1 (B), R33.2
- new net: D13.2 (A), R39.1
- new net: R46.2, U14.2 (CS)
- new net: C34.1, J11.1 (Pin_1), Q7.1, U14.6 (GND)
- new net: Q7.2, Q7.5
- new net: Q7.4, U14.3 (OC)
- new net: Q7.6, U14.1 (OD)
- new net: Q6.3 (C), R34.1
- new net: D15.2 (A), R41.1
- new net: J8.1 (Pin_1), U13.7 (OUT+)
- new net: D11.2 (A), R37.1
- new net: D12.2 (A), R38.1
- new net: C34.2, R45.2, U14.5 (VCC)
- new net: D17.2 (A), R43.1
- new net BACKLIGHT: J7.30 (Pin_30), R33.1, R35.1
- new net BAT+: J10.1 (Pin_1), J7.26 (Pin_26), J7.27 (Pin_27), J7.28 (Pin_28), R45.1
- new net FRONT_3V3: C33.1, J7.45 (Pin_45), J7.46 (Pin_46), J7.47 (Pin_47), J7.48 (Pin_48), R35.2, R36.2, R47.2, U11.10 (VDD), U11.12 (LEDA), U12.3 (VCC), U13.10 (VDD), U13.5 (EN), U13.6 (VDD/NC)
- new net FRONT_5V: J7.49 (Pin_49), J7.50 (Pin_50)
- new net FRONT_GND: C33.2, D11.1 (K), D12.1 (K), D13.1 (K), D14.1 (K), D15.1 (K), D16.1 (K), D17.1 (K), D18.1 (K), J7.21 (Pin_21), J7.22 (Pin_22), J7.23 (Pin_23), J7.24 (Pin_24), J7.25 (Pin_25), J7.3 (Pin_3), J7.4 (Pin_4), Q6.2 (E), Q7.3, R46.1, R48.2, R49.2, R50.2, U11.13 (GND), U11.8 (GND), U12.1 (GND), U13.8 (GND)
- new net GPIO10: J7.37 (Pin_37), R50.1
- new net GPIO11: J7.20 (Pin_20), R44.2
- new net GPIO12: J7.19 (Pin_19), R43.2
- new net GPIO13: J7.18 (Pin_18), R42.2
- new net GPIO14: J7.17 (Pin_17), R41.2
- new net GPIO15: J7.16 (Pin_16), R40.2
- new net GPIO16: J7.15 (Pin_15), R39.2
- new net GPIO17: J7.14 (Pin_14), R38.2
- new net GPIO18: J7.13 (Pin_13), R37.2
- new net GPIO19/USBD-: J7.12 (Pin_12)
- new net GPIO20/USBD+: J7.11 (Pin_11)
- new net GPIO21: J7.10 (Pin_10)
- new net GPIO27: J7.9 (Pin_9)
- new net GPIO3: J7.44 (Pin_44)
- new net GPIO33: J7.7 (Pin_7), U11.5 (RS)
- new net GPIO34: J7.6 (Pin_6), U11.7 (CS)
- new net GPIO35: J7.5 (Pin_5), U11.3 (SDA)
- new net GPIO36: J7.29 (Pin_29), U11.4 (SCL)
- new net GPIO38: J7.31 (Pin_31)
- new net GPIO39: J7.32 (Pin_32)
- new net GPIO4: J7.43 (Pin_43)
- new net GPIO40: J7.33 (Pin_33)
- new net GPIO41: J7.34 (Pin_34)
- new net GPIO42: J7.35 (Pin_35)
- new net GPIO45: J7.36 (Pin_36)
- new net GPIO47: J7.8 (Pin_8), R36.1, U11.6 (RESET), U12.2 (RESET)
- new net GPIO5/SDA: J7.42 (Pin_42), U13.3 (SDA)
- new net GPIO6/SCL: J7.41 (Pin_41), U13.2 (SCL)
- new net GPIO7: J7.40 (Pin_40), R47.1
- new net GPIO8: J7.39 (Pin_39), R48.1
- new net GPIO9: J7.38 (Pin_38), R49.1
- new net LEDK: R34.2, U11.11 (LEDK)
- new net U0RXD: J7.1 (Pin_1)
- new net U0TXD: J7.2 (Pin_2)
- no-connect marks 0 -> 5
Other:
- note added: "CUSTOM WATCH ADDRESS 4BIT WATCHFACE 1 = 0001"
- note added: "D/C & TFTRST ARE GPIO-CONTROLLED"
- note added: "LOWER RESISTOR VALUE AS NEEDED OR PWM CONTROL RANDOMIZED LED COLORS LED CURRENT = <18mA"
- company: (none) -> mechameka0
- title: (none) -> Faceplate: 0.96" SPI TFT + LED Array

Commit message: v1.2
WIP of major revisions of PCB board. Changed components and layout for better routing
Parts:
- Q6: value MMBT2222A -> MMBT2222ALT3G
Connections:
- net FRONT_5V: no longer names the net of J7.49 (Pin_49)
- net FRONT_5V: no longer J7.50 (Pin_50)
- no-connect marks 5 -> 7
Other:
- company: mechameka0 -> MECHAMEKA
- title: Faceplate: 0.96" SPI TFT + LED Array -> satWatch
Changed lines of the file:
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@@
 	(paper "A4")
 	(title_block
-		(title "Faceplate: 0.96\" SPI TFT + LED Array")
-		(rev "0")
-		(company "mechameka0")
+		(title "satWatch")
+		(rev "2.0")
+		(company "MECHAMEKA")
 		(comment 1 "Default watchface")
 	)
@@
 	)
 	(junction
-		(at 137.16 86.36)
-		(diameter 0)
-		(color 0 0 0 0)
-	)
-	(junction
 		(at 55.88 148.59)
 		(diameter 0)
@@
 	)
 	(no_connect
+		(at 134.62 86.36)
+	)
+	(no_connect
 		(at 251.46 40.64)
 	)
@@
 	)
 	(no_connect
+		(at 134.62 88.9)
+	)
+	(no_connect
 		(at 251.46 38.1)
 	)
@@
 	(wire
 		(pts
-			(xy 134.62 86.36) (xy 137.16 86.36)
-		)
-		(stroke
-			(width 0)
-			(type default)
-		)
-	)
-	(wire
-		(pts
 			(xy 58.42 53.34) (xy 64.77 53.34)
 		)
@@
 	(wire
 		(pts
-			(xy 137.16 88.9) (xy 134.62 88.9)
-		)
-		(stroke
-			(width 0)
-			(type default)
-		)
-	)
-	(wire
-		(pts
 			(xy 113.03 38.1) (xy 121.92 38.1)
 		)
@@
 	(wire
 		(pts
-			(xy 137.16 86.36) (xy 137.16 88.9)
-		)
-		(stroke
-			(width 0)
-			(type default)
-		)
-	)
-	(wire
-		(pts
 			(xy 66.04 68.58) (xy 58.42 68.58)
 		)
@@
 	(wire
 		(pts
-			(xy 146.05 86.36) (xy 137.16 86.36)
-		)
-		(stroke
-			(width 0)
-			(type default)
-		)
-	)
-	(wire
-		(pts
 			(xy 121.92 81.28) (xy 121.92 83.82)
 		)
@@
 	(symbol
 		(lib_id "power:+1V0")
-		(at 146.05 86.36 0)
-		(unit 1)
-		(body_style 1)
-		(exclude_from_sim no)
-		(in_bom yes)
-		(on_board yes)
-		(in_pos_files yes)
-		(dnp no)
-		(fields_autoplaced yes)
-		(property "Reference" "#PWR075"
-			(at 146.05 90.17 0)
-			(hide yes)
-			(show_name no)
-			(do_not_autoplace no)
-			(effects
-				(font
-					(size 1.27 1.27)
-				)
-			)
-		)
-		(property "Value" "FRONT_5V"
-			(at 146.05 81.28 0)
-			(show_name no)
-			(do_not_autoplace no)
-			(effects
-				(font
-					(size 1.27 1.27)
-				)
-			)
-		)
-		(property "Footprint" ""
-			(at 146.05 86.36 0)
-			(hide yes)
-			(show_name no)
-			(do_not_autoplace no)
-			(effects
-				(font
-					(size 1.27 1.27)
-				)
-			)
-		)
-		(property "Datasheet" ""
-			(at 146.05 86.36 0)
-			(hide yes)
-			(show_name no)
-			(do_not_autoplace no)
-			(effects
-				(font
-					(size 1.27 1.27)
-				)
-			)
-		)
-		(property "Description" "Power symbol creates a global label with name \"+1V0\""
-			(at 146.05 86.36 0)
-			(hide yes)
-			(show_name no)
-			(do_not_autoplace no)
-			(effects
-				(font
-					(size 1.27 1.27)
-				)
-			)
-		)
-		(pin "1"
-		)
-		(instances
-			(project "satWatch_main"
-				(path "/b975a3df-968d-424f-9025-993d668abad1/0425e4d7-ccce-4e74-a234-f8bc72f3ee67"
-					(reference "#PWR075")
-					(unit 1)
-				)
-			)
-		)
-	)
-	(symbol
-		(lib_id "power:+1V0")
 		(at 222.25 146.05 0)
 		(unit 1)
@@
 			)
 		)
-		(property "Value" "MMBT2222A"
+		(property "Value" "MMBT2222ALT3G"
 			(at 257.81 109.2199 0)
 			(show_name no)
