File: schematics/satWatch_main/satWatch_mainboard.kicad_sch (KiCad schematic)
At the start: 58 parts, among them J1 Conn_02x25_Top_Bottom, J2 Pogo_02x03_UARTPROG, Q1 DMP1045U, Q2 RE1C002UN, Q3 RE1C002UN, SW1 R-667995, SW2 R-667995, SW3 EVQ-P7A01P, SW4 EVQ-P7A01P, SW5 EVQ-P7A01P, U1 PAM2401SCADJ, U2 MIC5365-1.8YC5, U3 ESP32-S3-MINI-1, U4 MAX30101EFD_T, U5 BNO085, U6 DS3231MZ, Y1 32.768Hz

Commit message: v1.1
Completed board layout for charging dock configuration and a default watchface config
Parts:
- added C29: 0.1uF, Capacitor_SMD:C_0402_1005Metric_Pad0.74x0.62mm_HandSolder, symbol Device:C_Small
- added C30: 10uF, Capacitor_SMD:C_0402_1005Metric_Pad0.74x0.62mm_HandSolder, symbol Device:C_Small
- added C31, C32: 1uF, Capacitor_SMD:C_0402_1005Metric_Pad0.74x0.62mm_HandSolder, symbol Device:C_Small
- added D10: RED, LED_SMD:LED_0402_1005Metric_Pad0.77x0.64mm_HandSolder, symbol Device:LED
- added D8: DONE, LED_SMD:LED_0402_1005Metric_Pad0.77x0.64mm_HandSolder, symbol Device:LED
- added D9: CHRG, LED_SMD:LED_0402_1005Metric_Pad0.77x0.64mm_HandSolder, symbol Device:LED
- added J5, J6: SOLDER POINT, Connector_Wire:SolderWire-0.25sqmm_1x01_D0.65mm_OD1.7mm, symbol Connector:Conn_01x01_Pin
- added R29, R30: 1K, Resistor_SMD:R_0402_1005Metric_Pad0.72x0.64mm_HandSolder, symbol Device:R_US
- added R31: 1.2k, Resistor_SMD:R_0402_1005Metric_Pad0.72x0.64mm_HandSolder, symbol Device:R_US
- added R32: 5.1K(1%), Resistor_SMD:R_0402_1005Metric_Pad0.72x0.64mm_HandSolder, symbol Device:R_Small_US
- added U10: NCP186AMX330TAG, footprint:PSON40P160X120X45-9N, symbol import_symbol:NCP186AMX330TAG
- added U9: TP4056-42-ESOP8, Package_SO:SOIC-8-1EP_3.9x4.9mm_P1.27mm_EP2.41x3.3mm_ThermalVias, symbol Battery_Management:TP4056-42-ESOP8
- J1: value Conn_02x25_Top_Bottom -> 2167010509_MOLEX
- renumbered C13 to C12, C12 to C13, C16 to C15, C15 to C16, C19 to C17, C17 to C18, C20 to C19, C18 to C20, C4 to C3, C6 to C4, C8 to C5, C9 to C6, C3 to C8, C5 to C9, R8 to R10, R9 to R11, R10 to R12, R11 to R13, R17 to R14, R12 to R15, R13 to R6, R14 to R7, R6 to R8, R7 to R9
Connections:
- net BAT+: now also C30.1, U9.5 (BAT)
- net GND: now also C29.2, C30.2, C31.2, C32.2, D10.1 (K), J6.1 (Pin_1), R31.2, U10.5 (GND), U10.9 (EPAD), U9.1 (TEMP), U9.3 (GND), U9.9 (EPAD)
- net VIN_3V3: now also C32.1, R32.1, U10.1 (OUT), U10.2 (OUT__1), U10.4 (FB/ADJ)
- net GPIO35/BATTERY_MONITOR renamed BATTERY_MONITOR
- net BATTERY_MONITOR: now also U3.30 (IO48); no longer U3.31 (IO35)
- net GPIO48 renamed GPIO35
- net GPIO35: now also U3.31 (IO35); no longer U3.30 (IO48)
- net GPIO7/SCK renamed GPIO7
- net GPIO8/MISO renamed GPIO8
- net GPIO9/MOSI renamed GPIO9
- new net: D8.1 (K), R29.1
- new net: R29.2, U9.6 (~{STDBY})
- new net: D9.1 (K), R30.1
- new net: R31.1, U9.2 (PROG)
- new net: D10.2 (A), R32.2
- new net: R30.2, U9.7 (~{CHRG})
- new net VDOCK_5V: C29.1, C31.1, D8.2 (A), D9.2 (A), J5.1 (Pin_1), U10.6 (EN), U10.7 (IN), U10.8 (IN__1), U9.4 (V_{CC}), U9.8 (CE)
- no-connect marks 7 -> 8
Other:
- note added: "3.3V REGULATOR OUTPUT CURRENT: 1A QUIESCENT CURRENT: 140uA"
- note added: "MOUNTS TO AN EXTERNAL CHARGING DOCK BATTERY OVERCHARGE/DISCHARGE (DW01A) TYPICALLY INCLUDED IN FACEPLATE 1000mAh/1A"
- note added: "POPULATE ONLY FOR DOCKUNIT SETUP"
- moved on the sheet: BT1, C1, C10, C11, C12, C13, C14, C15, C16, C17, C18, C19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

Commit message: v1.2
WIP of major revisions of PCB board. Changed components and layout for better routing
Parts:
- removed H1, H2, H3: MountingHole, MountingHole:MountingHole_2.5mm, symbol Mechanical:MountingHole
- added C37: 1uF/6.3V, Capacitor_SMD:C_0402_1005Metric_Pad0.74x0.62mm_HandSolder, symbol Device:C_Small
- added C38: 10uF/6.3V, Capacitor_SMD:C_0402_1005Metric_Pad0.74x0.62mm_HandSolder, symbol Device:C_Small
- added U21: ADP5063, Package_DFN_QFN:QFN-20-1EP_4x4mm_P0.5mm_EP2.5x2.5mm, symbol Battery_Management:ADP5063
- added U22: AXP2101, Package_DFN_QFN:QFN-40-1EP_5x5mm_P0.4mm_EP3.6x3.6mm_ThermalVias, symbol symbols:AXP2101
Connections:
- net GND: now also C37.1, C38.1, U22.3 (GND), U22.40 (EP)
- new net: C37.2, U22.2 (VREF)
- new net: U21.10 (ISO_Sx), U21.11 (ISO_Sx), U21.9 (ISO_Sx)
- new net: U21.12 (ISO_Bx), U21.13 (ISO_Bx), U21.14 (ISO_Bx)
- new net: U21.6 (VINx), U21.7 (VINx), U21.8 (VINx)
- new net AXP2101_PWRON: U22.30 (PWRON)
- new net VUSB_5V: C38.2, U22.37 (VBUS)
Other:
- company: (none) -> MECHAMEKA
- title: (none) -> satWatch
- moved on the sheet: C7, C8, C9, Q2, Q3, R10, R11, R12, R13, R4, R5, R8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
