File: schematics/satWatch_main/satWatch_programmer.kicad_sch (KiCad schematic)
At the start: 35 parts, among them J3 855-22-006-10-001101, J4 UJ20-C-H-G-MSMT-2B-P16-TR, Q6 S8050, Q7 S8050, SW6 EVQ-P7A01P, SW7 EVQ-P7A01P, U7 CP2102N-Axx-xQFN28, U8 AMS1117-3.3

Commit message: v1.1
Completed board layout for charging dock configuration and a default watchface config
Parts:
- renumbered C25 to C21, C26 to C22, C27 to C23, C28 to C24, C21 to C25, C22 to C26, C23 to C27, C24 to C28, D4 to D2, D5 to D3, D2 to D4, D6 to D5, D7 to D6, D3 to D7, Q6 to Q4, Q7 to Q5, R15 to R16, R16 to R17, R28 to R18, R20 to R19, R18 to R20, R19 to R21, R21 to R22, R24 to R23, R26 to R24, R22 to R25, R23 to R26, R25 to R27, R27 to R28

Commit message: v1.2
WIP of major revisions of PCB board. Changed components and layout for better routing
Other:
- company: mechameka -> MECHAMEKA
- title: UART Programmer Board -> satWatch
Changed lines of the file:
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@@
 	(paper "A4")
 	(title_block
-		(title "UART Programmer Board")
-		(rev "V0")
-		(company "mechameka")
+		(title "satWatch")
+		(rev "2.0")
+		(company "MECHAMEKA")
 		(comment 1 "Component reference from ESP32-S3 DevKitC")
 	)
