File: schematics/proteus_watch/face1.kicad_sch (KiCad schematic)
At the start: 41 parts, among them J10 BAT+, J11 BAT-, J7 2167010509_MOLEX, J8 MOTOR+, J9 MOTOR-, Q6 MMBT2222ALT3G, Q7 FS8205, U14 DRV2605LDGS, U15 DW01A

Commit message: v1.31
wip integrating face3
Connections:
- net GPIO48: now reaches J7.38 (Pin_38), R50.1
Changed lines of the file:
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@@
+		)
+	)
+	(label "GPIO48"
+		(at 133.35 58.42 0)
+		(effects
+			(font
+				(size 1.27 1.27)
+			)
+			(justify left bottom)
 		)
 	)
