File: schematics/proteus_watch/mainboard.kicad_sch (KiCad schematic)
At the start: 69 parts, among them J1 2167010509_MOLEX, J2 SOLDER PAD, J3 SOLDER PAD, Q2 RE1C002UN, Q3 RE1C002UN, SW1 R-667995, SW2 R-667995, SW3 EVQ-P7A01P, SW4 EVQ-P7A01P, SW5 EVQ-P7A01P, U1 MAX17048G+T10, U10 LSM6DSO, U11 BQ25185, U3 MIC2876-5.0YMT-TR, U4 MIC5365-1.8YMT-TZ, U5 NCP186AMX330TAG, U6 ESP32-S3-MINI-1, U7 MAX30101EFD_T, U8 PCF85063ATL, Y1 32.768kHZ, 7pF, 60kOhms

Commit message: v1.3
progress update with PCB layout. Repurposing old board design.
Other:
- note added: "LiPo BATTERY CHARGER AND POWER PATH MANAGEMENT INPUT CHARGE LIMIT = 1.1A BATTERY VOLTAGE = 4.2V CHARGE CURRENT = 300/R.ISET (A) CHARGE CURRENT = 483mA STAT1: LOW ON FAULT STAT2: LOW ON CHARGING BAT_NTC = 10K(25C) BETA(25/85)= 3435K NTC"
- note removed: "LiPo BATTERY CHARGER AND POWER PATH MANAGEMENT INPUT CHARGE LIMIT = 1.1A BATTERY VOLTAGE = 4.2V CHARGE CURRENT = 300/R.ISET (A) CHARGE CURRENT = 483mA STAT1: LOW ON FAULT STAT2: LOW ON CHARGING BAT_NTC = 10K(25C) BETA(3435K) NTC"
Changed lines of the file:
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@@
 		)
 	)
-	(text "LiPo BATTERY CHARGER AND POWER PATH MANAGEMENT\n\nINPUT CHARGE LIMIT = 1.1A\nBATTERY VOLTAGE = 4.2V\nCHARGE CURRENT = 300/R.ISET (A)\n	CHARGE CURRENT = 483mA\n\nSTAT1: LOW ON FAULT\nSTAT2: LOW ON CHARGING\n\nBAT_NTC = 10K(25C) BETA(3435K) NTC"
+	(text "LiPo BATTERY CHARGER AND POWER PATH MANAGEMENT\n\nINPUT CHARGE LIMIT = 1.1A\nBATTERY VOLTAGE = 4.2V\nCHARGE CURRENT = 300/R.ISET (A)\n	CHARGE CURRENT = 483mA\n\nSTAT1: LOW ON FAULT\nSTAT2: LOW ON CHARGING\n\nBAT_NTC = 10K(25C) BETA(25/85)= 3435K NTC"
 		(exclude_from_sim no)
 		(at 17.018 29.464 0)
@@
 			(justify right bottom)
 		)
-		(property "Net Class" ""
+		(property "Netclass" ""
 			(at 140.97 201.93 0)
 			(show_name no)
@@
 			(justify right bottom)
 		)
-		(property "Net Class" ""
+		(property "Netclass" ""
 			(at 140.97 204.47 0)
 			(show_name no)
@@
 			(justify right bottom)
 		)
-		(property "Net Class" ""
+		(property "Netclass" ""
 			(at 158.75 81.28 0)
 			(show_name no)
@@
 			(justify right bottom)
 		)
-		(property "Net Class" ""
+		(property "Netclass" ""
 			(at 158.75 78.74 0)
 			(show_name no)
